File: 2A/Detection_PCB/detection_pcb/detection_pcb.kicad_pcb (KiCad board)
At the start: 2 copper layers, 96 x 96 mm, 141 parts, among them J1 BAT, Q1 PMOS, U1 VL53L1X_module, U10 VL53L1X_module, U11 VL53L1X_module, U12 VL53L1X_module, U13 VL53L1X_module, U14 VL53L1X_module, U15 VL53L1X_module, U16 VL53L1X_module, U17 Buck_3.3V, U18 STM32G070, U2 VL53L1X_module, U3 VL53L1X_module, U4 VL53L1X_module, U5 VL53L1X_module, U6 VL53L1X_module, U7 VL53L1X_module, U8 VL53L1X_module, U9 VL53L1X_module, Y1 16MHz

Commit message: detection V2.1
Parts:
- added XSDN11: TestPoint, TestPoint:TestPoint_Pad_D1.0mm, B.Cu at (130.5, 114.2)
- renumbered XSDN6 to XSDN1, XSDN9 to XSDN10, XSDN14 to XSDN12, XSDN12 to XSDN13, XSDN5 to XSDN14, XSDN3 to XSDN15, XSDN1 to XSDN16, XSDN15 to XSDN2, XSDN13 to XSDN3, XSDN11 to XSDN4, XSDN8 to XSDN5, XSDN7 to XSDN6, XSDN2 to XSDN7, XSDN10 to XSDN8, XSDN4 to XSDN9
Connections:
- R12 pad 1: XSDN4 -> XSDN5
- R13 pad 1: XSDN5 -> XSDN6
- R16 pad 1: XSDN6 -> XSDN7
- R17 pad 1: XSDN7 -> XSDN8
- R20 pad 1: XSDN8 -> XSDN9
- R21 pad 1: XSDN9 -> XSDN10
- R24 pad 1: XSDN10 -> XSDN11
- R25 pad 1: XSDN11 -> XSDN12
- R28 pad 1: XSDN12 -> XSDN13
- R29 pad 1: XSDN13 -> XSDN14
- R3 pad 1: XSDN0 -> XSDN1
- R32 pad 1: XSDN14 -> XSDN15
- R33 pad 1: XSDN15 -> XSDN16
- R4 pad 1: XSDN1 -> XSDN2
- R7 pad 1: XSDN2 -> XSDN3
- R8 pad 1: XSDN3 -> XSDN4
- U1 pad 3: XSDN0 -> XSDN1
- U10 pad 3: XSDN9 -> XSDN10
- U11 pad 3: XSDN10 -> XSDN11
- U12 pad 3: XSDN11 -> XSDN12
- U13 pad 3: XSDN12 -> XSDN13
- U14 pad 3: XSDN13 -> XSDN14
- U15 pad 3: XSDN14 -> XSDN15
- U16 pad 3: XSDN15 -> XSDN16
- U18 pad 15: XSDN0 -> XSDN1
- U18 pad 2: XSDN2 -> XSDN3
- U18 pad 21: XSDN15 -> XSDN16
- U18 pad 24: XSDN14 -> XSDN15
- U18 pad 27: XSDN13 -> XSDN14
- U18 pad 30: XSDN12 -> XSDN13
- U18 pad 33: XSDN11 -> XSDN12
- U18 pad 36: XSDN10 -> XSDN11
- U18 pad 37: LED10 -> SCL
- U18 pad 39: XSDN9 -> XSDN10
- U18 pad 43: SCL -> LED10
- U18 pad 44: XSDN8 -> XSDN9
- U18 pad 49: XSDN7 -> XSDN8
- U18 pad 5: XSDN1 -> XSDN2
- U18 pad 52: XSDN6 -> XSDN7
- U18 pad 57: XSDN5 -> XSDN6
- U18 pad 60: XSDN4 -> XSDN5
- U18 pad 63: XSDN3 -> XSDN4
- U2 pad 3: XSDN1 -> XSDN2
- U3 pad 3: XSDN2 -> XSDN3
- U4 pad 3: XSDN3 -> XSDN4
- U5 pad 3: XSDN4 -> XSDN5
- U6 pad 3: XSDN5 -> XSDN6
- U7 pad 3: XSDN6 -> XSDN7
- U8 pad 3: XSDN7 -> XSDN8
- U9 pad 3: XSDN8 -> XSDN9
- XSDN1 pad 1: XSDN0 -> XSDN1
- XSDN10 pad 1: XSDN9 -> XSDN10
- XSDN12 pad 1: XSDN11 -> XSDN12
- XSDN13 pad 1: XSDN12 -> XSDN13
- XSDN14 pad 1: XSDN13 -> XSDN14
- XSDN15 pad 1: XSDN14 -> XSDN15
- XSDN16 pad 1: XSDN15 -> XSDN16
- XSDN2 pad 1: XSDN1 -> XSDN2
- XSDN3 pad 1: XSDN2 -> XSDN3
- XSDN4 pad 1: XSDN3 -> XSDN4
- XSDN5 pad 1: XSDN4 -> XSDN5
- XSDN6 pad 1: XSDN5 -> XSDN6
- XSDN7 pad 1: XSDN6 -> XSDN7
- XSDN8 pad 1: XSDN7 -> XSDN8
- XSDN9 pad 1: XSDN8 -> XSDN9
Routing:
- net XSDN16: track 0.00 -> 42.4 mm
- net XSDN0: track 41.5 -> 0.00 mm
- net SCL: track 274.9 -> 264.4 mm, vias 17 -> 19
- net LED10: track 40.6 -> 47.9 mm, vias 1 -> 5
- net XSDN15: track 42.4 -> 49.4 mm
- net XSDN14: track 49.4 -> 42.7 mm
- net XSDN5: track 43.5 -> 38.5 mm
- net XSDN3: track 38.6 -> 43.5 mm
- net SDA: track 251.7 -> 246.9 mm
- net XSDN9: track 39.6 -> 44.1 mm
- net XSDN2: track 43.5 -> 39.3 mm
- net XSDN13: track 42.7 -> 38.9 mm
- net XSDN8: track 44.1 -> 40.6 mm
- net XSDN10: track 43.0 -> 39.6 mm
- net XSDN12: track 38.9 -> 41.5 mm
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Other:
- board text added: "detection v2.1"
- board text removed: "detection v2"
