File: 2A/Detection_PCB/detection_pcb/mcu.kicad_sch (KiCad schematic)
At the start: 35 parts, among them U18 STM32G070, Y1 16MHz

Commit message: detection V2.1
Parts:
- added XSDN11: TestPoint, TestPoint:TestPoint_Pad_D1.0mm, symbol Connector:TestPoint
- renumbered XSDN6 to XSDN1, XSDN9 to XSDN10, XSDN14 to XSDN12, XSDN12 to XSDN13, XSDN5 to XSDN14, XSDN3 to XSDN15, XSDN1 to XSDN16, XSDN15 to XSDN2, XSDN13 to XSDN3, XSDN11 to XSDN4, XSDN8 to XSDN5, XSDN7 to XSDN6, XSDN2 to XSDN7, XSDN10 to XSDN8, XSDN4 to XSDN9
Connections:
- net XSDN0 is gone; now on net XSDN1: U18.15 (PC2), XSDN1.1
- net LED10: now also U18.43 (PA11); no longer U18.37 (PA9)
- net SCL: now also U18.37 (PA9); no longer U18.43 (PA11)
- net XSDN1: no longer U18.5 (PC15), XSDN2.1
- net XSDN10: now also U18.39 (PC7), XSDN10.1; no longer U18.36 (PA8)
- net XSDN11: now also U18.36 (PA8), XSDN11.1; no longer U18.33 (PB13), XSDN12.1
- net XSDN12: now also U18.33 (PB13), XSDN12.1; no longer U18.30 (PB10), XSDN13.1
- net XSDN13: now also U18.30 (PB10), XSDN13.1; no longer U18.27 (PB0), XSDN14.1
- net XSDN14: now also U18.27 (PB0), XSDN14.1; no longer U18.24 (PA7), XSDN15.1
- net XSDN15: now also U18.24 (PA7), XSDN15.1; no longer U18.21 (PA4), XSDN16.1
- net XSDN2: now also U18.5 (PC15), XSDN2.1; no longer U18.2 (PC12), XSDN3.1
- net XSDN3: now also U18.2 (PC12), XSDN3.1; no longer U18.63 (PB9), XSDN4.1
- net XSDN4: now also U18.63 (PB9), XSDN4.1; no longer U18.60 (PB6), XSDN5.1
- net XSDN5: now also U18.60 (PB6), XSDN5.1; no longer U18.57 (PB3), XSDN6.1
- net XSDN6: now also U18.57 (PB3), XSDN6.1; no longer U18.52 (PD2), XSDN7.1
- net XSDN7: now also U18.52 (PD2), XSDN7.1; no longer U18.49 (PC9), XSDN8.1
- net XSDN8: now also U18.49 (PC9), XSDN8.1; no longer U18.44 (PA12), XSDN9.1
- net XSDN9: now also U18.44 (PA12), XSDN9.1; no longer U18.39 (PC7), XSDN10.1
- new net XSDN16: U18.21 (PA4), XSDN16.1
Other:
- note added: "XSDN1 = PC2 XSDN2 = PC15 XSDN3 = PC12 XSDN4 = PB9 XSDN5 = PB6 XSDN6 = PB3 XSDN7 = PD2 XSDN8 = PC9 XSDN9 = PA12 XSDN10 = PC7 XSDN11 = PA8 XSDN12 = PB13 XSDN13 = PB10 XSDN14 = PB0 XSDN15 = PA7 XSDN16 = PA4"
- note removed: "XSDN0 = PC2 XSDN1 = PC15 XSDN2 = PC12 XSDN3 = PB9 XSDN4 = PB6 XSDN5 = PB3 XSDN6 = PD2 XSDN7 = PC9 XSDN8 = PA12 XSDN9 = PC7 XSDN10 = PA8 XSDN11 = PB13 XSDN12 = PB10 XSDN13 = PB0 XSDN14 = PA7 XSDN15 = PA4"
