File: 2A/Detection_PCB/detection_pcb/sensors.kicad_sch (KiCad schematic)
At the start: 64 parts, among them U1 VL53L1X_module, U10 VL53L1X_module, U11 VL53L1X_module, U12 VL53L1X_module, U13 VL53L1X_module, U14 VL53L1X_module, U15 VL53L1X_module, U16 VL53L1X_module, U2 VL53L1X_module, U3 VL53L1X_module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

Commit message: detection V2.1
Connections:
- net XSDN0 is gone; now on net XSDN1: R3.1, U1.3 (XSDN)
- net XSDN1: no longer R4.1, U2.3 (XSDN)
- net XSDN10: now also R21.1, U10.3 (XSDN); no longer R24.1, U11.3 (XSDN)
- net XSDN11: now also R24.1, U11.3 (XSDN); no longer R25.1, U12.3 (XSDN)
- net XSDN12: now also R25.1, U12.3 (XSDN); no longer R28.1, U13.3 (XSDN)
- net XSDN13: now also R28.1, U13.3 (XSDN); no longer R29.1, U14.3 (XSDN)
- net XSDN14: now also R29.1, U14.3 (XSDN); no longer R32.1, U15.3 (XSDN)
- net XSDN15: now also R32.1, U15.3 (XSDN); no longer R33.1, U16.3 (XSDN)
- net XSDN2: now also R4.1, U2.3 (XSDN); no longer R7.1, U3.3 (XSDN)
- net XSDN3: now also R7.1, U3.3 (XSDN); no longer R8.1, U4.3 (XSDN)
- net XSDN4: now also R8.1, U4.3 (XSDN); no longer R12.1, U5.3 (XSDN)
- net XSDN5: now also R12.1, U5.3 (XSDN); no longer R13.1, U6.3 (XSDN)
- net XSDN6: now also R13.1, U6.3 (XSDN); no longer R16.1, U7.3 (XSDN)
- net XSDN7: now also R16.1, U7.3 (XSDN); no longer R17.1, U8.3 (XSDN)
- net XSDN8: now also R17.1, U8.3 (XSDN); no longer R20.1, U9.3 (XSDN)
- net XSDN9: now also R20.1, U9.3 (XSDN); no longer R21.1, U10.3 (XSDN)
- new net XSDN16: R33.1, U16.3 (XSDN)
