File: 2A/Com/NUCELO64_ESP32_HAT/NUCELO64_ESP32_HAT.kicad_pcb (KiCad board)
At the start: 2 copper layers, 57.4 x 33.4 mm, 2 parts

Commit message: majPCB
Parts:
- U1: renamed from _; value uPesy ESP32 Wroom -> uPesy_ESP32_Wroom_DevKit
Connections:
- U1 pad 29: unconnected-(U1-Pad29) -> /WIFI_STATE
- XA1 pad A3: unconnected-(XA1-PadA3) -> /WIFI_STATE
Routing:
- net /WIFI_STATE: track 0.00 -> 19.8 mm
Changed lines of the file:
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@@
   (net 5 "unconnected-(U1-Pad30)")
   (net 6 "unconnected-(U1-Pad3)")
-  (net 7 "unconnected-(U1-Pad29)")
+  (net 7 "/WIFI_STATE")
   (net 8 "unconnected-(U1-Pad4)")
   (net 9 "unconnected-(U1-Pad28)")
@@
   (net 33 "unconnected-(XA1-PadA1)")
   (net 34 "unconnected-(XA1-PadA2)")
-  (net 35 "unconnected-(XA1-PadA3)")
-  (net 36 "unconnected-(XA1-PadA4)")
-  (net 37 "unconnected-(XA1-PadA5)")
-  (net 38 "unconnected-(XA1-PadD0)")
-  (net 39 "unconnected-(XA1-PadD1)")
-  (net 40 "unconnected-(XA1-PadD3)")
-  (net 41 "unconnected-(XA1-PadD4)")
-  (net 42 "unconnected-(XA1-PadD5)")
-  (net 43 "unconnected-(XA1-PadD6)")
-  (net 44 "unconnected-(XA1-PadD7)")
-  (net 45 "unconnected-(XA1-PadD8)")
-  (net 46 "unconnected-(XA1-PadD9)")
-  (net 47 "unconnected-(XA1-PadVIN)")
+  (net 35 "unconnected-(XA1-PadA4)")
+  (net 36 "unconnected-(XA1-PadA5)")
+  (net 37 "unconnected-(XA1-PadD0)")
+  (net 38 "unconnected-(XA1-PadD1)")
+  (net 39 "unconnected-(XA1-PadD3)")
+  (net 40 "unconnected-(XA1-PadD4)")
+  (net 41 "unconnected-(XA1-PadD5)")
+  (net 42 "unconnected-(XA1-PadD6)")
+  (net 43 "unconnected-(XA1-PadD7)")
+  (net 44 "unconnected-(XA1-PadD8)")
+  (net 45 "unconnected-(XA1-PadD9)")
+  (net 46 "unconnected-(XA1-PadVIN)")
   (footprint "arduino Boards:Arduino_Uno_Shield" (layer "F.Cu")
     (at 101.6 57.957881 -90)
@@
       (net 34 "unconnected-(XA1-PadA2)") (pinfunction "A2") (pintype "bidirectional"))
     (pad "A3" thru_hole oval (at 58.42 -2.54 270) (size 1.7272 1.7272) (drill 1.016) (layers *.Cu *.Mask)
-      (net 35 "unconnected-(XA1-PadA3)") (pinfunction "A3") (pintype "bidirectional"))
+      (net 7 "/WIFI_STATE") (pinfunction "A3") (pintype "bidirectional"))
     (pad "A4" thru_hole oval (at 60.96 -2.54 270) (size 1.7272 1.7272) (drill 1.016) (layers *.Cu *.Mask)
-      (net 36 "unconnected-(XA1-PadA4)") (pinfunction "A4") (pintype "bidirectional"))
+      (net 35 "unconnected-(XA1-PadA4)") (pinfunction "A4") (pintype "bidirectional"))
     (pad "A5" thru_hole oval (at 63.5 -2.54 270) (size 1.7272 1.7272) (drill 1.016) (layers *.Cu *.Mask)
-      (net 37 "unconnected-(XA1-PadA5)") (pinfunction "A5") (pintype "bidirectional"))
+      (net 36 "unconnected-(XA1-PadA5)") (pinfunction "A5") (pintype "bidirectional"))
     (pad "D0" thru_hole oval (at 63.5 -50.8 270) (size 1.7272 1.7272) (drill 1.016) (layers *.Cu *.Mask)
-      (net 38 "unconnected-(XA1-PadD0)") (pinfunction "D0_RX0") (pintype "bidirectional"))
+      (net 37 "unconnected-(XA1-PadD0)") (pinfunction "D0_RX0") (pintype "bidirectional"))
     (pad "D1" thru_hole oval (at 60.96 -50.8 270) (size 1.7272 1.7272) (drill 1.016) (layers *.Cu *.Mask)
-      (net 39 "unconnected-(XA1-PadD1)") (pinfunction "D1_TX0") (pintype "bidirectional"))
+      (net 38 "unconnected-(XA1-PadD1)") (pinfunction "D1_TX0") (pintype "bidirectional"))
     (pad "D2" thru_hole oval (at 58.42 -50.8 270) (size 1.7272 1.7272) (drill 1.016) (layers *.Cu *.Mask)
       (net 15 "/USART1_RX") (pinfunction "D2_INT0") (pintype "bidirectional"))
     (pad "D3" thru_hole oval (at 55.88 -50.8 270) (size 1.7272 1.7272) (drill 1.016) (layers *.Cu *.Mask)
-      (net 40 "unconnected-(XA1-PadD3)") (pinfunction "D3_INT1") (pintype "bidirectional"))
+      (net 39 "unconnected-(XA1-PadD3)") (pinfunction "D3_INT1") (pintype "bidirectional"))
     (pad "D4" thru_hole oval (at 53.34 -50.8 270) (size 1.7272 1.7272) (drill 1.016) (layers *.Cu *.Mask)
-      (net 41 "unconnected-(XA1-PadD4)") (pinfunction "D4") (pintype "bidirectional"))
+      (net 40 "unconnected-(XA1-PadD4)") (pinfunction "D4") (pintype "bidirectional"))
     (pad "D5" thru_hole oval (at 50.8 -50.8 270) (size 1.7272 1.7272) (drill 1.016) (layers *.Cu *.Mask)
-      (net 42 "unconnected-(XA1-PadD5)") (pinfunction "D5") (pintype "bidirectional"))
+      (net 41 "unconnected-(XA1-PadD5)") (pinfunction "D5") (pintype "bidirectional"))
     (pad "D6" thru_hole oval (at 48.26 -50.8 270) (size 1.7272 1.7272) (drill 1.016) (layers *.Cu *.Mask)
-      (net 43 "unconnected-(XA1-PadD6)") (pinfunction "D6") (pintype "bidirectional"))
+      (net 42 "unconnected-(XA1-PadD6)") (pinfunction "D6") (pintype "bidirectional"))
     (pad "D7" thru_hole oval (at 45.72 -50.8 270) (size 1.7272 1.7272) (drill 1.016) (layers *.Cu *.Mask)
-      (net 44 "unconnected-(XA1-PadD7)") (pinfunction "D7") (pintype "bidirectional"))
+      (net 43 "unconnected-(XA1-PadD7)") (pinfunction "D7") (pintype "bidirectional"))
     (pad "D8" thru_hole oval (at 41.656 -50.8 270) (size 1.7272 1.7272) (drill 1.016) (layers *.Cu *.Mask)
-      (net 45 "unconnected-(XA1-PadD8)") (pinfunction "D8") (pintype "bidirectional"))
+      (net 44 "unconnected-(XA1-PadD8)") (pinfunction "D8") (pintype "bidirectional"))
     (pad "D9" thru_hole oval (at 39.116 -50.8 270) (size 1.7272 1.7272) (drill 1.016) (layers *.Cu *.Mask)
-      (net 46 "unconnected-(XA1-PadD9)") (pinfunction "D9") (pintype "bidirectional"))
+      (net 45 "unconnected-(XA1-PadD9)") (pinfunction "D9") (pintype "bidirectional"))
     (pad "D10" thru_hole oval (at 36.576 -50.8 270) (size 1.7272 1.7272) (drill 1.016) (layers *.Cu *.Mask)
       (net 13 "/USART1_TX") (pinfunction "D10_CS") (pintype "bidirectional"))
@@
       (net 1 "GND") (pinfunction "GND") (pintype "power_in"))
     (pad "VIN" thru_hole oval (at 45.72 -2.54 270) (size 1.7272 1.7272) (drill 1.016) (layers *.Cu *.Mask)
-      (net 47 "unconnected-(XA1-PadVIN)") (pinfunction "VIN") (pintype "power_in"))
+      (net 46 "unconnected-(XA1-PadVIN)") (pinfunction "VIN") (pintype "power_in"))
   )
   (footprint "uPesy Boards:uPesy_ESP32_Wroom_DevKit" (layer "F.Cu")
@@
     (property "Sheetname" "")
     (attr through_hole)
-    (fp_text reference "_" (at 0 -19.4 90) (layer "F.SilkS")
-      (effects (font (size 1 1) (thickness 0.15)))
-    )
-    (fp_text value "uPesy ESP32 Wroom" (at -0.04 0) (layer "F.Fab")
+    (fp_text reference "U1" (at 0 -19.4 90) (layer "F.SilkS")
+      (effects (font (size 1 1) (thickness 0.15)))
+    )
+    (fp_text value "uPesy_ESP32_Wroom_DevKit" (at -0.04 0) (layer "F.Fab")
       (effects (font (size 1 1) (thickness 0.15)))
     )
@@
       (net 9 "unconnected-(U1-Pad28)") (pinfunction "GPIO0") (pintype "bidirectional"))
     (pad "29" thru_hole circle (at 11.4954 11.4938) (size 1.7 1.7) (drill 1) (layers *.Cu *.Mask)
-      (net 7 "unconnected-(U1-Pad29)") (pinfunction "GPIO2") (pintype "bidirectional"))
+      (net 7 "/WIFI_STATE") (pinfunction "GPIO2") (pintype "bidirectional"))
     (pad "30" thru_hole circle (at 11.4954 14.0338) (size 1.7 1.7) (drill 1) (layers *.Cu *.Mask)
       (net 5 "unconnected-(U1-Pad30)") (pinfunction "GPIO15") (pintype "bidirectional"))
@@
   (segment (start 104.14 98.597881) (end 108.873219 98.597881) (width 0.5) (layer "F.Cu") (net 1))
   (segment (start 104.14 101.137881) (end 104.14 98.597881) (width 0.5) (layer "F.Cu") (net 1))
+  (segment (start 107.68 120.68) (end 107.68 118.37) (width 0.5) (layer "F.Cu") (net 7))
+  (segment (start 117.58 121.85) (end 108.85 121.85) (width 0.5) (layer "F.Cu") (net 7))
+  (segment (start 118.4462 120.9838) (end 117.58 121.85) (width 0.5) (layer "F.Cu") (net 7))
+  (segment (start 108.85 121.85) (end 107.68 120.68) (width 0.5) (layer "F.Cu") (net 7))
+  (segment (start 105.687881 116.377881) (end 104.14 116.377881) (width 0.5) (layer "F.Cu") (net 7))
+  (segment (start 118.4462 119.4954) (end 118.4462 120.9838) (width 0.5) (layer "F.Cu") (net 7))
+  (segment (start 107.68 118.37) (end 105.687881 116.377881) (width 0.5) (layer "F.Cu") (net 7))
   (segment (start 152.4 94.533881) (end 150.56 96.373881) (width 0.5) (layer "F.Cu") (net 13))
   (segment (start 150.56 97.84) (end 149.73 98.67) (width 0.5) (layer "F.Cu") (net 13))
