File: 2A/Com/NUCELO64_ESP32_HAT/NUCELO64_ESP32_HAT.kicad_sch (KiCad schematic)
At the start: 2 parts, among them U1 uPesy_ESP32_Wroom_DevKit

Commit message: majPCB
Connections:
- net WIFI_STATE: now reaches U1.29 (GPIO2)
- net WIFI_STATE: now also XA1.A3
Changed lines of the file:
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@@
+    (stroke (width 0) (type default) (color 0 0 0 0))
+  )
+  (wire (pts (xy 219.71 96.52) (xy 228.6 96.52))
     (stroke (width 0) (type default) (color 0 0 0 0))
   )
@@
     (stroke (width 0) (type default) (color 0 0 0 0))
   )
+  (wire (pts (xy 59.69 90.17) (xy 64.77 90.17))
+    (stroke (width 0) (type default) (color 0 0 0 0))
+  )
   (wire (pts (xy 130.81 113.03) (xy 140.97 113.03))
     (stroke (width 0) (type default) (color 0 0 0 0))
@@
     (effects (font (size 1.27 1.27)) (justify left bottom))
   )
+  (label "WIFI_STATE" (at 228.6 96.52 0)
+    (effects (font (size 1.27 1.27)) (justify left bottom))
+  )
+  (label "WIFI_STATE" (at 59.69 90.17 0)
+    (effects (font (size 1.27 1.27)) (justify left bottom))
+  )
