File: 1A/Cherrycount/PCB/CherrycountPCB.kicad_sch (KiCad schematic)
At the start: 22 parts, among them J1 Conn_01x02_Female, J2 Conn_01x03_Female, J3 Conn_01x05_Female, J4 Screw_Terminal_01x02, J5 Screw_Terminal_01x02, Q1 2SA1015, Q2 2SA1015

Commit message: Version finale du PCB de compteur de cerises
Parts:
- added J4: Screw_Terminal_01x02, TerminalBlock:TerminalBlock_bornier-2_P5.08mm, symbol Connector:Screw_Terminal_01x02
- renumbered J4 to J5, J5 to J6
Connections:
- net at J5.1 (Pin_1): now also J4.1 (Pin_1); no longer F1.1
- new net: F1.1, J4.2 (Pin_2)
Other:
- moved on the sheet: D1, F1, J5, J6

Commit message: Version finale du PCB de compteur de cerises
Connections:
- net GND: now also J3.5 (Pin_5); no longer J3.4 (Pin_4)
- net VIN: now also J3.4 (Pin_4); no longer J3.5 (Pin_5)
Changed lines of the file:
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@@
     )
   )
-  (global_label "VIN" (shape input) (at 60.96 71.12 0) (fields_autoplaced)
+  (global_label "VIN" (shape input) (at 60.96 73.66 0) (fields_autoplaced)
     (effects (font (size 1.27 1.27)) (justify left))
-    (property "Références Inter-Feuilles" "${INTERSHEET_REFS}" (id 0) (at 66.3969 71.0406 0)
+    (property "Références Inter-Feuilles" "${INTERSHEET_REFS}" (id 0) (at 66.3969 73.5806 0)
       (effects (font (size 1.27 1.27)) (justify left) hide)
     )
@@
     (pin "2")
   )
-  (symbol (lib_id "power:GND") (at 60.96 73.66 90) (unit 1)
+  (symbol (lib_id "power:GND") (at 60.96 71.12 90) (unit 1)
     (in_bom yes) (on_board yes) (fields_autoplaced)
-    (property "Reference" "#PWR04" (id 0) (at 67.31 73.66 0)
+    (property "Reference" "#PWR04" (id 0) (at 67.31 71.12 0)
       (effects (font (size 1.27 1.27)) hide)
     )
-    (property "Value" "GND" (id 1) (at 64.77 73.6599 90)
+    (property "Value" "GND" (id 1) (at 64.77 71.1199 90)
       (effects (font (size 1.27 1.27)) (justify right))
     )
-    (property "Footprint" "" (id 2) (at 60.96 73.66 0)
+    (property "Footprint" "" (id 2) (at 60.96 71.12 0)
       (effects (font (size 1.27 1.27)) hide)
     )
-    (property "Datasheet" "" (id 3) (at 60.96 73.66 0)
+    (property "Datasheet" "" (id 3) (at 60.96 71.12 0)
       (effects (font (size 1.27 1.27)) hide)
     )

Commit message: Correction du code Arduino & PCB Cherrycount
Parts:
- removed A1: Arduino_UNO_R3, Module:Arduino_UNO_R3, symbol MCU_Module:Arduino_UNO_R3
- removed Q1, Q2: 2SA1015, Package_TO_SOT_THT:TO-92_Inline, symbol Transistor_BJT:2SA1015
- added A1: Arduino_Leonardo, Module:Arduino_UNO_R3, symbol MCU_Module:Arduino_Leonardo
- added Q1, Q2: S8550, Package_TO_SOT_THT:TO-92_Inline, symbol Transistor_BJT:S8550
- D1: value DIODE -> ${SIM.PARAMS}; Spice_Netlist_Enabled Y -> (none); Spice_Primitive D -> (none)
Connections:
- net BASE1: now also A1.22 (D7)
- net BASE2: now also A1.23 (D8)
- net Conn1x3: now also A1.16 (D1/TX)
- net D12: now also A1.27 (D12)
- net D6: now also A1.21 (D6)
- net GND: now also A1.6 (GND)
- net VIN: now also A1.8 (VIN)
- net at AFF1.10 (g), AFF2.10 (g), R7.2: no longer AFF1.2 (d), AFF2.2 (d), R4.2
- net at AFF2.3 (C.A.): now also Q2.3 (C)
- net at AFF1.3 (C.A.): now also Q1.3 (C)
- net at R9.2: now also Q1.2 (B)
- net at R3.1: now also A1.19 (D4)
- net at R8.1: now also A1.28 (D13)
- net at R2.1: now also A1.17 (D2/SDA)
- net at R1.1: now also A1.18 (D3/SCL)
- net at R4.1: now also A1.20 (D5)
- net at R7.1: now also A1.24 (D9)
- net at R5.1: now also A1.25 (D10)
- net at R6.1: now also A1.26 (D11)
- net at J3.3 (Pin_3): now also A1.5 (+5V), Q1.1 (E), Q2.1 (E); no longer J1.1 (Pin_1)
- net at R10.2: now also Q2.2 (B)
- new net: AFF1.2 (d), AFF2.2 (d), R4.2
- new net: A1.15 (D0/RX), J1.1 (Pin_1)
- no-connect marks 17 -> 16
Other:
- moved on the sheet: J1

Commit message: Correction du code Arduino & PCB Cherrycount
Parts:
- added R11: 1M, Resistor_SMD:R_0805_2012Metric_Pad1.20x1.40mm_HandSolder, symbol Device:R
Connections:
- net GND: now also R11.1
- net at A1.15 (D0/RX), J1.1 (Pin_1): now also R11.2
Other:
- moved on the sheet: J1
Changed lines of the file:
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@@
   (junction (at 189.23 72.39) (diameter 0) (color 0 0 0 0)
+  )
+  (junction (at 69.85 41.91) (diameter 0) (color 0 0 0 0)
   )
   (junction (at 185.42 74.93) (diameter 0) (color 0 0 0 0)
@@
     (stroke (width 0) (type default))
   )
+  (wire (pts (xy 69.85 41.91) (xy 118.11 41.91))
+    (stroke (width 0) (type default))
+  )
   (wire (pts (xy 195.58 109.22) (xy 185.42 109.22))
     (stroke (width 0) (type default))
   )
-  (wire (pts (xy 60.96 50.8) (xy 118.11 50.8))
+  (wire (pts (xy 60.96 41.91) (xy 69.85 41.91))
     (stroke (width 0) (type default))
   )
@@
     (stroke (width 0) (type default))
   )
-  (wire (pts (xy 118.11 50.8) (xy 118.11 80.01))
+  (wire (pts (xy 118.11 41.91) (xy 118.11 80.01))
     (stroke (width 0) (type default))
   )
@@
     )
   )
-  (symbol (lib_id "power:GND") (at 60.96 48.26 90) (unit 1)
-    (in_bom yes) (on_board yes) (dnp no) (fields_autoplaced)
-    (property "Reference" "#PWR02" (at 67.31 48.26 0)
-      (effects (font (size 1.27 1.27)) hide)
-    )
-    (property "Value" "GND" (at 64.77 48.2599 90)
+  (symbol (lib_id "power:GND") (at 60.96 39.37 90) (unit 1)
+    (in_bom yes) (on_board yes) (dnp no) (fields_autoplaced)
+    (property "Reference" "#PWR02" (at 67.31 39.37 0)
+      (effects (font (size 1.27 1.27)) hide)
+    )
+    (property "Value" "GND" (at 64.77 39.3699 90)
       (effects (font (size 1.27 1.27)) (justify right))
     )
-    (property "Footprint" "" (at 60.96 48.26 0)
-      (effects (font (size 1.27 1.27)) hide)
-    )
-    (property "Datasheet" "" (at 60.96 48.26 0)
+    (property "Footprint" "" (at 60.96 39.37 0)
+      (effects (font (size 1.27 1.27)) hide)
+    )
+    (property "Datasheet" "" (at 60.96 39.37 0)
       (effects (font (size 1.27 1.27)) hide)
     )
@@
         (path "/ec662bfd-1d68-47f9-bb5f-35a9f3e1bc4d"
           (reference "AFF1") (unit 1)
+        )
+      )
+    )
+  )
+  (symbol (lib_id "Device:R") (at 69.85 45.72 180) (unit 1)
+    (in_bom yes) (on_board yes) (dnp no) (fields_autoplaced)
+    (property "Reference" "R11" (at 72.39 45.085 0)
+      (effects (font (size 1.27 1.27)) (justify right))
+    )
+    (property "Value" "1M" (at 72.39 47.625 0)
+      (effects (font (size 1.27 1.27)) (justify right))
+    )
+    (property "Footprint" "Resistor_SMD:R_0805_2012Metric_Pad1.20x1.40mm_HandSolder" (at 71.628 45.72 90)
+      (effects (font (size 1.27 1.27)) hide)
+    )
+    (property "Datasheet" "~" (at 69.85 45.72 0)
+      (effects (font (size 1.27 1.27)) hide)
+    )
+    (pin "1")
+    (pin "2")
+    (instances
+      (project "CherrycountPCB"
+        (path "/ec662bfd-1d68-47f9-bb5f-35a9f3e1bc4d"
+          (reference "R11") (unit 1)
         )
       )
@@
     )
   )
-  (symbol (lib_id "Connector:Conn_01x02_Female") (at 55.88 50.8 180) (unit 1)
-    (in_bom yes) (on_board yes) (dnp no) (fields_autoplaced)
-    (property "Reference" "J1" (at 54.61 50.8001 0)
+  (symbol (lib_id "power:GND") (at 69.85 49.53 0) (unit 1)
+    (in_bom yes) (on_board yes) (dnp no) (fields_autoplaced)
+    (property "Reference" "#PWR07" (at 69.85 55.88 0)
+      (effects (font (size 1.27 1.27)) hide)
+    )
+    (property "Value" "GND" (at 69.85 54.61 0)
+      (effects (font (size 1.27 1.27)))
+    )
+    (property "Footprint" "" (at 69.85 49.53 0)
+      (effects (font (size 1.27 1.27)) hide)
+    )
+    (property "Datasheet" "" (at 69.85 49.53 0)
+      (effects (font (size 1.27 1.27)) hide)
+    )
+    (pin "1")
+    (instances
+      (project "CherrycountPCB"
+        (path "/ec662bfd-1d68-47f9-bb5f-35a9f3e1bc4d"
+          (reference "#PWR07") (unit 1)
+        )
+      )
+    )
+  )
+  (symbol (lib_id "Connector:Conn_01x02_Female") (at 55.88 41.91 180) (unit 1)
+    (in_bom yes) (on_board yes) (dnp no) (fields_autoplaced)
+    (property "Reference" "J1" (at 54.61 41.9101 0)
       (effects (font (size 1.27 1.27)) (justify left))
     )
-    (property "Value" "Conn_01x02_Female" (at 54.61 48.2601 0)
+    (property "Value" "Conn_01x02_Female" (at 54.61 39.3701 0)
       (effects (font (size 1.27 1.27)) (justify left))
     )
-    (property "Footprint" "Connector_PinHeader_2.54mm:PinHeader_1x02_P2.54mm_Vertical" (at 55.88 50.8 0)
-      (effects (font (size 1.27 1.27)) hide)
-    )
-    (property "Datasheet" "~" (at 55.88 50.8 0)
-      (effects (font (size 1.27 1.27)) hide)
-    )
+    (property "Footprint" "Connector_PinHeader_2.54mm:PinHeader_1x02_P2.54mm_Vertical" (at 55.88 41.91 0)
+      (effects (font (size 1.27 1.27)) hide)
+    )
+    (property "Datasheet" "~" (at 55.88 41.91 0)
+      (effects (font (size 1.27 1.27)) hide)
+    )

Commit message: Code final Cherrycount/ajout fichier step ax12
Parts:
- J4, J5, J6: footprint TerminalBlock:TerminalBlock_bornier-2_P5.08mm -> 7seg:180G-2-vertical
Connections:
- net GND: no longer J1.2 (Pin_2)
- net VIN: no longer J2.2 (Pin_2)
- net at J1.1 (Pin_1), R11.2: now also A1.14 (A5); no longer A1.15 (D0/RX)
- net at A1.5 (+5V), J3.3 (Pin_3), Q1.1 (E)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: now also J1.2 (Pin_2), J2.2 (Pin_2)
Changed lines of the file:
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@@
   (junction (at 189.23 72.39) (diameter 0) (color 0 0 0 0)
   )
+  (junction (at 185.42 74.93) (diameter 0) (color 0 0 0 0)
+  )
+  (junction (at 173.99 107.95) (diameter 0) (color 0 0 0 0)
+  )
+  (junction (at 167.64 116.84) (diameter 0) (color 0 0 0 0)
+  )
+  (junction (at 97.79 60.96) (diameter 0) (color 0 0 0 0)
+  )
+  (junction (at 193.04 69.85) (diameter 0) (color 0 0 0 0)
+  )
+  (junction (at 261.62 90.17) (diameter 0) (color 0 0 0 0)
+  )
+  (junction (at 180.34 99.06) (diameter 0) (color 0 0 0 0)
+  )
   (junction (at 69.85 41.91) (diameter 0) (color 0 0 0 0)
   )
-  (junction (at 185.42 74.93) (diameter 0) (color 0 0 0 0)
-  )
-  (junction (at 173.99 107.95) (diameter 0) (color 0 0 0 0)
-  )
-  (junction (at 167.64 116.84) (diameter 0) (color 0 0 0 0)
-  )
-  (junction (at 193.04 69.85) (diameter 0) (color 0 0 0 0)
-  )
-  (junction (at 261.62 90.17) (diameter 0) (color 0 0 0 0)
-  )
-  (junction (at 180.34 99.06) (diameter 0) (color 0 0 0 0)
-  )
   (junction (at 74.93 101.6) (diameter 0) (color 0 0 0 0)
   )
@@
   (junction (at 182.88 77.47) (diameter 0) (color 0 0 0 0)
   )
+  (no_connect (at 90.17 113.03))
   (no_connect (at 90.17 95.25))
-  (no_connect (at 90.17 113.03))
   (no_connect (at 220.98 104.14))
   (no_connect (at 100.33 123.19))
@@
   (no_connect (at 90.17 97.79))
   (no_connect (at 90.17 90.17))
-  (no_connect (at 90.17 107.95))
   (no_connect (at 90.17 100.33))
   (no_connect (at 105.41 123.19))
+  (no_connect (at 115.57 80.01))
   (no_connect (at 100.33 69.85))
   (no_connect (at 90.17 115.57))
@@
     (stroke (width 0) (type default))
   )
+  (wire (pts (xy 60.96 60.96) (xy 97.79 60.96))
+    (stroke (width 0) (type default))
+  )
   (wire (pts (xy 157.48 88.9) (xy 167.64 88.9))
     (stroke (width 0) (type default))
@@
     (stroke (width 0) (type default))
   )
+  (wire (pts (xy 97.79 39.37) (xy 97.79 53.34))
+    (stroke (width 0) (type default))
+  )
   (wire (pts (xy 173.99 107.95) (xy 173.99 116.84))
     (stroke (width 0) (type default))
@@
     (stroke (width 0) (type default))
   )
-  (wire (pts (xy 97.79 53.34) (xy 97.79 69.85))
+  (wire (pts (xy 97.79 53.34) (xy 97.79 60.96))
     (stroke (width 0) (type default))
   )
@@
     (stroke (width 0) (type default))
   )
+  (wire (pts (xy 60.96 39.37) (xy 97.79 39.37))
+    (stroke (width 0) (type default))
+  )
   (wire (pts (xy 74.93 102.87) (xy 74.93 101.6))
     (stroke (width 0) (type default))
@@
     (stroke (width 0) (type default))
   )
+  (wire (pts (xy 86.36 41.91) (xy 86.36 107.95))
+    (stroke (width 0) (type default))
+  )
   (wire (pts (xy 97.79 53.34) (xy 269.24 53.34))
     (stroke (width 0) (type default))
@@
     (stroke (width 0) (type default))
   )
-  (wire (pts (xy 69.85 41.91) (xy 118.11 41.91))
-    (stroke (width 0) (type default))
-  )
   (wire (pts (xy 195.58 109.22) (xy 185.42 109.22))
     (stroke (width 0) (type default))
@@
     (stroke (width 0) (type default))
   )
-  (wire (pts (xy 118.11 80.01) (xy 115.57 80.01))
-    (stroke (width 0) (type default))
-  )
   (wire (pts (xy 76.2 53.34) (xy 97.79 53.34))
     (stroke (width 0) (type default))
@@
     (stroke (width 0) (type default))
   )
+  (wire (pts (xy 97.79 60.96) (xy 97.79 69.85))
+    (stroke (width 0) (type default))
+  )
   (wire (pts (xy 180.34 114.3) (xy 195.58 114.3))
     (stroke (width 0) (type default))
   )
-  (wire (pts (xy 118.11 41.91) (xy 118.11 80.01))
-    (stroke (width 0) (type default))
-  )
   (wire (pts (xy 157.48 107.95) (xy 173.99 107.95))
     (stroke (width 0) (type default))
@@
     (stroke (width 0) (type default))
   )
+  (wire (pts (xy 86.36 107.95) (xy 90.17 107.95))
+    (stroke (width 0) (type default))
+  )
   (wire (pts (xy 185.42 109.22) (xy 185.42 74.93))
     (stroke (width 0) (type default))
   )
+  (wire (pts (xy 69.85 41.91) (xy 86.36 41.91))
+    (stroke (width 0) (type default))
+  )
   (wire (pts (xy 163.83 72.39) (xy 189.23 72.39))
     (stroke (width 0) (type default))
@@
     )
     (property "Références Inter-Feuilles" "${INTERSHEET_REFS}" (at 65.8526 78.6606 0)
-      (effects (font (size 1.27 1.27)) (justify left) hide)
-    )
-  )
-  (global_label "VIN" (shape input) (at 60.96 60.96 0) (fields_autoplaced)
-    (effects (font (size 1.27 1.27)) (justify left))
-    (property "Intersheetrefs" "${INTERSHEET_REFS}" (at 0 0 0)
-      (effects (font (size 1.27 1.27)) hide)
-    )
-    (property "Références Inter-Feuilles" "${INTERSHEET_REFS}" (at 66.3969 60.8806 0)
       (effects (font (size 1.27 1.27)) (justify left) hide)
     )
@@
       (effects (font (size 1.27 1.27)))
     )
-    (property "Footprint" "TerminalBlock:TerminalBlock_bornier-2_P5.08mm" (at 48.26 101.6 0)
+    (property "Footprint" "7seg:180G-2-vertical" (at 48.26 101.6 0)
       (effects (font (size 1.27 1.27)) hide)
     )
@@
         (path "/ec662bfd-1d68-47f9-bb5f-35a9f3e1bc4d"
           (reference "#PWR03") (unit 1)
-        )
-      )
-    )
-  )
-  (symbol (lib_id "power:GND") (at 60.96 39.37 90) (unit 1)
-    (in_bom yes) (on_board yes) (dnp no) (fields_autoplaced)
-    (property "Reference" "#PWR02" (at 67.31 39.37 0)
-      (effects (font (size 1.27 1.27)) hide)
-    )
-    (property "Value" "GND" (at 64.77 39.3699 90)
-      (effects (font (size 1.27 1.27)) (justify right))
-    )
-    (property "Footprint" "" (at 60.96 39.37 0)
-      (effects (font (size 1.27 1.27)) hide)
-    )
-    (property "Datasheet" "" (at 60.96 39.37 0)
-      (effects (font (size 1.27 1.27)) hide)
-    )
-    (pin "1")
-    (instances
-      (project "CherrycountPCB"
-        (path "/ec662bfd-1d68-47f9-bb5f-35a9f3e1bc4d"
-          (reference "#PWR02") (unit 1)
         )
       )
@@
       (effects (font (size 1.27 1.27)))
     )
-    (property "Footprint" "TerminalBlock:TerminalBlock_bornier-2_P5.08mm" (at 57.15 96.52 0)
+    (property "Footprint" "7seg:180G-2-vertical" (at 57.15 96.52 0)
       (effects (font (size 1.27 1.27)) hide)
     )
@@
       (effects (font (size 1.27 1.27)))
     )
-    (property "Footprint" "TerminalBlock:TerminalBlock_bornier-2_P5.08mm" (at 48.26 118.11 0)
-      (effects (font (size 1.27 1.27)) hide)
-    )
+    (property "Footprint" "7seg:180G-2-vertical" (at 48.26 118.11 0)
+      (effects (font (size 1.27 1.27)) hide)
+    )
